File: hardware/nrfmicro.kicad_sch (KiCad schematic)
At the start: 24 parts, among them J1 USB-C USB 2.0 MC-372, J2 Conn_01x04, J3 Conn_01x02, J4 Conn_01x04, Q1 AO3407, Q2 AO3407, U1 E73-2G4M08S1C, U2 AP2112K-3.3, U3 TP4054, U4 ProMicro, X1 32768kHz

Commit message: bmd-340 variant: start
Parts:
- removed J4: Conn_01x04, nrfmicro:connector_usb, symbol Connector_Generic:Conn_01x04
- removed U1: E73-2G4M08S1C, nrfmicro:E73-2G4M08S1C-52840, symbol nrfmicro:E73-2G4M08S1C-52840
- added U5: BMD-340, nrfmicro:BMD-340, symbol Rigado:BMD-340
Connections:
- net BATTERY_PIN: now also U5.20 (P0.04/AIN2)
- net BLUE_LED: now also U5.53 (P1.10)
- net DATA+: now also U5.68 (USB-D+)
- net DATA-: now also U5.67 (USB-D-)
- net GND: now also U5.1 (GND), U5.16 (GND), U5.18 (GND), U5.2 (GND), U5.29 (GND), U5.3 (GND), U5.30 (GND), U5.4 (GND), U5.45 (GND), U5.46 (GND), U5.47 (GND), U5.5 (GND), U5.55 (GND)
- net P0.00: now also U5.13 (P0.00/XTAL1)
- net P0.01: now also U5.14 (P0.01/XTAL2)
- net P0.02: now also U5.15 (P0.02/AIN0)
- net P0.03: now also U5.19 (P0.03/AIN1)
- net P0.06: now also U5.22 (P0.06)
- net P0.07: now also U5.23 (P0.07/TRACECLK)
- net P0.08: now also U5.24 (P0.08)
- net P0.09: now also U5.25 (P0.09/NFC1)
- net P0.10: now also U5.26 (P0.10/NFC2)
- net P0.12: now also U5.28 (P0.12/TRACEDATA[1])
- net P0.13: now also U5.31 (P0.13)
- net P0.15: now also U5.33 (P0.15)
- net P0.17: now also U5.35 (P0.17)
- net P0.20: now also U5.38 (P0.20)
- net P0.22: now also U5.40 (P0.22)
- net P0.24: now also U5.42 (P0.24)
- net P0.26: now also U5.7 (P0.26)
- net P0.28: now also U5.9 (P0.28/AIN4)
- net P0.29: now also U5.10 (P0.29/AIN5)
- net P0.30: now also U5.11 (P0.30/AIN6)
- net P0.31: now also U5.12 (P0.31/AIN7)
- net P1.00: now also U5.56 (SWO/TRACEDATA[0]/P1.00)
- net P1.02: now also U5.58 (P1.02)
- net P1.04: now also U5.60 (P1.04)
- net P1.06: now also U5.49 (P1.06)
- net P1.11: now also U5.54 (P1.11)
- net P1.13: now also U5.62 (P1.13)
- net POWER_PIN: now also U5.52 (TRACEDATA[3]/P1.09)
- net PROG: now also U5.21 (P0.05/AIN3)
- net RESET: now also U5.39 (P0.18/nRESET)
- net SWC: now also U5.43 (SWCLK)
- net SWD: now also U5.44 (SWDIO)
- net VBUS: now also U5.66 (VBUS)
- net nRF_VDD: now also U5.17 (VCC), U5.65 (VCCH)
Other:
- moved on the sheet: X1
